File: usbtele.sch (KiCad schematic (older format))
At the start: 11 parts, among them P1 USB_A, P2 CONN_01X03, U1 FT232RL

Commit message: Add Rev 1.0
Parts:
- D1, D2: symbol LED -> LED-RESCUE-usbtele
- P1: symbol USB_A -> USB_A-RESCUE-usbtele
Changed lines of the file:
@@
 EESchema Schematic File Version 2
+LIBS:usbtele-rescue
 LIBS:power
 LIBS:device
@@
 encoding utf-8
 Sheet 1 1
-Title ""
-Date "2016-12-15"
+Title "USB FrSky SmartPort adapter"
+Date "2016-12-28"
 Rev "1.0"
 Comp ""
@@
 Comment2 ""
 Comment3 ""
-Comment4 ""
+Comment4 "https://github.com/mirkix/USBtele"
 $EndDescr
 $Comp
@@
 $EndComp
 $Comp
-L USB_A P1
+L USB_A-RESCUE-usbtele P1
 U 1 1 5841DF82
 P 3650 3200
@@
 	7350 2600 7350 2750
 $Comp
-L LED D1
+L LED-RESCUE-usbtele D1
 U 1 1 5852604F
 P 7350 3450
@@
 $EndComp
 $Comp
-L LED D2
+L LED-RESCUE-usbtele D2
 U 1 1 585260C4
 P 7750 3450
